Commit message: urdf: rewrite humanoid_v2 to 20-DOF with arms, ankle_roll, fixed wrists
- Add full arm chain: shoulder_pitch/roll + elbow_pitch × 2 (SG92R ×4)
- Add ankle_roll joints + ankle_pitch_link intermediate links (MG996R ×4)
- Change wrist_pitch to fixed joints (крюк/заглушка, no servo)
- Fix left/right_knee_pitch axis 1→-1 (anatomically correct backward bend)
- Update HLD Hardware v1.4→v1.5: remove wrist DOF, fix weight ~1kg, 20 DOF

Co-Authored-By: Claude Sonnet 4.6 <noreply@anthropic.com>

File: Research/robot-research-vault/research/robot-hardware-research/artefacts/urdf/humanoid_v2.urdf (robot description, URDF)
Before this commit: robot roboforge_humanoid_v2, 24 links, 23 joints
Links:
- removed link camera_link
- removed link left_forearm
- removed link right_forearm
- added link left_lower_arm, mass 0.040; collision cylinder length=0.050 radius=0.010; visual cylinder length=0.050 radius=0.010
- added link right_lower_arm, mass 0.040; collision cylinder length=0.050 radius=0.010; visual cylinder length=0.050 radius=0.010
- link head: mass 0.030 -> 0.050
- link head_yaw_link: mass 0.005 -> 0.009
- link left_ankle_pitch_link: mass 0.010 -> 0.055
- link left_foot: geometry collision box size=0.025 0.065 0.010; visual box size=0.025 0.065 0.010
- link left_hand: mass 0.010 -> 0.015; geometry collision box size=0.018 0.012 0.030; visual box size=0.018 0.012 0.030
- link left_hip_roll_link: mass 0.010 -> 0.055
- link left_hip_yaw_link: mass 0.010 -> 0.055
- link left_lower_leg: mass 0.055 -> 0.100
- link left_shoulder_pitch_link: mass 0.005 -> 0.009
- link left_upper_arm: mass 0.025 -> 0.050; geometry collision cylinder length=0.055 radius=0.012; visual cylinder length=0.055 radius=0.012
- link left_upper_leg: mass 0.055 -> 0.100
- link right_ankle_pitch_link: mass 0.010 -> 0.055
- link right_foot: geometry collision box size=0.025 0.065 0.010; visual box size=0.025 0.065 0.010
- link right_hand: mass 0.010 -> 0.015; geometry collision box size=0.018 0.012 0.030; visual box size=0.018 0.012 0.030
- link right_hip_roll_link: mass 0.010 -> 0.055
- link right_hip_yaw_link: mass 0.010 -> 0.055
- link right_lower_leg: mass 0.055 -> 0.100
- link right_shoulder_pitch_link: mass 0.005 -> 0.009
- link right_upper_arm: mass 0.025 -> 0.050; geometry collision cylinder length=0.055 radius=0.012; visual cylinder length=0.055 radius=0.012
- link right_upper_leg: mass 0.055 -> 0.100
- link torso: mass 0.120 -> 0.250; geometry collision box size=0.06 0.04 0.12; visual box size=0.06 0.04 0.12
Joints:
- removed joint camera_joint
- joint head_pan: limit lower=-1.047 upper=1.047 effort=0.196 velocity=3.14 -> lower=-1.047 upper=1.047 effort=0.245 velocity=5.5; origin xyz=0 0 0.06 rpy=0 0 0 -> xyz=0 0 0.07 rpy=0 0 0
- joint head_tilt: limit lower=-0.524 upper=0.524 effort=0.196 velocity=3.14 -> lower=-0.524 upper=0.524 effort=0.245 velocity=5.5; origin xyz=0 0 0 rpy=0 0 0 -> xyz=0 0 0.025 rpy=0 0 0
- joint left_ankle_roll: limit lower=-0.349 upper=0.349 effort=0.980 velocity=3.14 -> lower=-0.524 upper=0.524 effort=0.980 velocity=3.14; origin xyz=0 0 0 rpy=0 0 0 -> xyz=0 0 -0.005 rpy=0 0 0
- joint left_elbow_pitch: axis 0 1 0 -> 1 0 0; child left_forearm -> left_lower_arm; limit lower=0 upper=2.094 effort=0.245 velocity=3.14 -> lower=0 upper=2.094 effort=0.245 velocity=5.5; origin xyz=0 0 -0.045 rpy=0 0 0 -> xyz=0 0 -0.055 rpy=0 0 0
- joint left_hip_pitch: origin xyz=0 0 -0.010 rpy=0 0 0 -> xyz=0 0 -0.020 rpy=0 0 0
- joint left_hip_roll: origin xyz=0 0 0 rpy=0 0 0 -> xyz=0 0 -0.030 rpy=0 0 0
- joint left_hip_yaw: origin xyz=0.025 0 -0.045 rpy=0 0 0 -> xyz=0.025 0 -0.065 rpy=0 0 0
- joint left_knee_pitch: axis 1 0 0 -> -1 0 0
- joint left_shoulder_pitch: axis 0 1 0 -> 1 0 0; limit lower=-1.571 upper=1.571 effort=0.245 velocity=3.14 -> lower=-1.571 upper=1.571 effort=0.245 velocity=5.5; origin xyz=0.045 0 0.03 rpy=0 0 0 -> xyz=0.035 0 0.040 rpy=0 0 0
- joint left_shoulder_roll: axis 1 0 0 -> 0 1 0; limit lower=-1.047 upper=1.047 effort=0.245 velocity=3.14 -> lower=-1.047 upper=1.047 effort=0.245 velocity=5.5; origin xyz=0 0 0 rpy=0 0 0 -> xyz=0 0 -0.010 rpy=0 0 0
- joint left_wrist_pitch: axis 0 1 0 -> (none); limit lower=-0.785 upper=0.785 effort=0.196 velocity=3.14 -> (none); origin xyz=0 0 -0.040 rpy=0 0 0 -> xyz=0 0 -0.050 rpy=0 0 0; parent left_forearm -> left_lower_arm; type revolute -> fixed
- joint right_ankle_roll: limit lower=-0.349 upper=0.349 effort=0.980 velocity=3.14 -> lower=-0.524 upper=0.524 effort=0.980 velocity=3.14; origin xyz=0 0 0 rpy=0 0 0 -> xyz=0 0 -0.005 rpy=0 0 0
- joint right_elbow_pitch: axis 0 1 0 -> 1 0 0; child right_forearm -> right_lower_arm; limit lower=0 upper=2.094 effort=0.245 velocity=3.14 -> lower=0 upper=2.094 effort=0.245 velocity=5.5; origin xyz=0 0 -0.045 rpy=0 0 0 -> xyz=0 0 -0.055 rpy=0 0 0
- joint right_hip_pitch: origin xyz=0 0 -0.010 rpy=0 0 0 -> xyz=0 0 -0.020 rpy=0 0 0
- joint right_hip_roll: origin xyz=0 0 0 rpy=0 0 0 -> xyz=0 0 -0.030 rpy=0 0 0
- joint right_hip_yaw: origin xyz=-0.025 0 -0.045 rpy=0 0 0 -> xyz=-0.025 0 -0.065 rpy=0 0 0
- joint right_shoulder_pitch: axis 0 1 0 -> 1 0 0; limit lower=-1.571 upper=1.571 effort=0.245 velocity=3.14 -> lower=-1.571 upper=1.571 effort=0.245 velocity=5.5; origin xyz=-0.045 0 0.03 rpy=0 0 0 -> xyz=-0.035 0 0.040 rpy=0 0 0
- joint right_shoulder_roll: axis 1 0 0 -> 0 1 0; limit lower=-1.047 upper=1.047 effort=0.245 velocity=3.14 -> lower=-1.047 upper=1.047 effort=0.245 velocity=5.5; origin xyz=0 0 0 rpy=0 0 0 -> xyz=0 0 -0.010 rpy=0 0 0
- joint right_wrist_pitch: axis 0 1 0 -> (none); limit lower=-0.785 upper=0.785 effort=0.196 velocity=3.14 -> (none); origin xyz=0 0 -0.040 rpy=0 0 0 -> xyz=0 0 -0.050 rpy=0 0 0; parent right_forearm -> right_lower_arm; type revolute -> fixed
